Commit message: Fix finger collision geom

File: thor_vt_hand_description/urdf/vt_finger_tud_single_link.urdf.xacro (robot description, xacro)
@@ -54,5 +54,6 @@
       </collision>
       <collision>
-        <origin xyz="-0.002 0.007 0.018" rpy="0 0 0"/>
+        <!--<origin xyz="0 -0.00407 0.04983" rpy="0.4 0 0"/>-->
+        <origin xyz="${-0.002+0.003} ${0.007-0.00407-0.005} ${0.018+0.04983} " rpy="0.4 0 0"/>
         <geometry>
           <cylinder length="0.05" radius="0.008"/>
