Commit message: Switch to using fixed joint instead of mimic

File: thor_vt_hand_description/urdf/vt_finger_tud.urdf.xacro (robot description, xacro)
@@ -82,4 +82,5 @@
 		<!-- joint list -->
 		<!-- WARNING: UPPER LIMIT NOT CORRECT/IGNORED WHILE USING MIMIC JOINT TYPE -->
+                <!--
                 <joint name="${prefix}_j1" type="revolute">
 			<parent link="${prefix}_link_0"/>
@@ -90,4 +91,13 @@
 			<mimic joint="${prefix}_j0" multiplier="0.4" offset="0"/>
 		</joint>
+		-->
+		<joint name="${prefix}_j1" type="fixed">
+                        <parent link="${prefix}_link_0"/>
+                        <child link="${prefix}_link_1"/>
+                        <axis xyz="1 0 0"/>
+                        <origin xyz="0 -0.00407 0.04983" rpy="0.4 0 0"/>
+                        <limit lower="0" upper="0.8" effort="100" velocity="100"/>
+                        <!--<mimic joint="${prefix}_j0" multiplier="0.4" offset="0"/>-->
+                </joint>
 		<!-- end of joint list -->
 	</xacro:macro>

Commit message: Use params inspired by Sandia hand to improve grasping quality

File: thor_vt_hand_description/urdf/vt_finger_tud.urdf.xacro (robot description, xacro)
@@ -1,4 +1,4 @@
 <!--
-paramter:
+parameters:
         prefix:         typcially includes the hand prefix and an identifier for the finger(i.e. finger_1, etc...).
         reflect:        finger0: reflect = 1
@@ -9,27 +9,27 @@
         <xacro:include filename="$(find thor_mang_description)/urdf/constants.xacro" />
         <xacro:macro name="vt_finger_tud_macro" params="prefix reflect">
-		<!-- link list -->
-		<link name="${prefix}_link_0">
-			<visual>
-				<origin xyz="0 0 0" rpy="0 0 0"/>
-				<geometry>
-					<mesh filename="package://thor_vt_hand_description/meshes/collision/${prefix}_link_0.stl" />
-				</geometry>
-				<material name="green">
-					<color rgba="0 1 0 1"/>
-				</material>
-			</visual>
-			<collision>
-				<origin xyz="0 0 0" rpy="0 ${M_PI*0.5} 0"/>
-                                 <geometry>
+                <!-- link list -->
+                <link name="${prefix}_link_0">
+                        <visual>
+                                <origin xyz="0 0 0" rpy="0 0 0"/>
+                                <geometry>
+                                        <mesh filename="package://thor_vt_hand_description/meshes/collision/${prefix}_link_0.stl" />
+                                </geometry>
+                                <material name="green">
+                                        <color rgba="0 1 0 1"/>
+                                </material>
+                        </visual>
+                        <collision>
+                                <origin xyz="0 0 0" rpy="0 ${M_PI*0.5} 0"/>
+                                <geometry>
                                     <cylinder length="0.02" radius="0.017" />
                                   </geometry>
-				<material name="yellow">
-					<color rgba="0 1 1 1"/>
-				</material>
-			</collision>
-			<collision>
+                                <material name="yellow">
+                                        <color rgba="0 1 1 1"/>
+                                </material>
+                        </collision>
+                        <collision>
                                 <origin xyz="0 0 0.02" rpy="0 0 0"/>
-                                 <geometry>
+                                <geometry>
                                     <cylinder length="0.04" radius="0.008" />
                                   </geometry>
@@ -38,5 +38,5 @@
                         <collision>
                                 <origin xyz="0 -0.00407 0.042" rpy="0 ${M_PI*0.5} 0"/>
-                                 <geometry>
+                                <geometry>
                                     <cylinder length="0.02" radius="0.014" />
                                   </geometry>
@@ -45,5 +45,5 @@
                                 </material>
                         </collision>
-	    <!-- WARNING: INERTIA NOT CORRECT -->
+            <!-- WARNING: INERTIA NOT CORRECT -->
             <inertial>
                 <origin xyz="${reflect*0.2e-03} 0.92e-03 21.11e-03" rpy="0 0 0"/>
@@ -51,22 +51,32 @@
                 <inertia ixx="21.39e-06" ixy="${reflect*(-0.39e-06)}" ixz="${reflect*0.71e-06}" iyy="18.98e-06" iyz="-1.36e-06" izz="4.73e-06" />
             </inertial>
-		</link>
-		<link name="${prefix}_link_1">
-			<visual>
-				<origin xyz="0 0 0" rpy="0 0 0"/>
-				<geometry>
-					<mesh filename="package://thor_vt_hand_description/meshes/collision/${prefix}_link_1.stl" />
-				</geometry>
-				<material name="green"/>
-			</visual>
-			<collision>
-				<origin xyz="-0.002 0.007 0.018" rpy="0 0 0"/>
-                                 <geometry>
+                </link>
+                    <gazebo reference="${prefix}_link_0">
+      <mu1>1.1</mu1>
+      <mu2>1.1</mu2>
+      <kp>1000000.0</kp>
+      <kd>10.0</kd>
+      <maxVel>0.1</maxVel>
+      <minDepth>0.00</minDepth>
+      <maxContacts>1</maxContacts>
+      <!--<material>Gazebo/FlatBlack</material>-->
+    </gazebo>
+                <link name="${prefix}_link_1">
+                        <visual>
+                                <origin xyz="0 0 0" rpy="0 0 0"/>
+                                <geometry>
+                                        <mesh filename="package://thor_vt_hand_description/meshes/collision/${prefix}_link_1.stl" />
+                                </geometry>
+                                <material name="green"/>
+                        </visual>
+                        <collision>
+                                <origin xyz="-0.002 0.007 0.018" rpy="0 0 0"/>
+                                <geometry>
                                     <cylinder length="0.05" radius="0.008" />
                                   </geometry>
-				<material name="yellow"/>
-			</collision>
-	    <!-- WARNING: INERTIA NOT CORRECT -->
-	    <!--
+                                <material name="yellow"/>
+                        </collision>
+            <!-- WARNING: INERTIA NOT CORRECT -->
+            <!--
             <inertial>
                 <origin xyz="${reflect*-0.99e-03} -4.42e-03 11.82e-03" rpy="0 0 0"/>
@@ -78,19 +88,29 @@
               <origin xyz="0.0 0.005 0.02" rpy="0 0 0"/>
             </xacro:inertial_cuboid__with_pose_macro>
-		</link>
-		<!-- end of link list -->
-		<!-- joint list -->
-		<!-- WARNING: UPPER LIMIT NOT CORRECT/IGNORED WHILE USING MIMIC JOINT TYPE -->
+                </link>
+                    <gazebo reference="${prefix}_link_1">
+      <mu1>1.1</mu1>
+      <mu2>1.1</mu2>
+      <kp>1000000.0</kp>
+      <kd>10.0</kd>
+      <maxVel>0.1</maxVel>
+      <minDepth>0.00</minDepth>
+      <maxContacts>1</maxContacts>
+      <!--<material>Gazebo/FlatBlack</material>-->
+    </gazebo>
+                <!-- end of link list -->
+                <!-- joint list -->
+                <!-- WARNING: UPPER LIMIT NOT CORRECT/IGNORED WHILE USING MIMIC JOINT TYPE -->
                 <!--
                 <joint name="${prefix}_j1" type="revolute">
-			<parent link="${prefix}_link_0"/>
-			<child link="${prefix}_link_1"/>
-			<axis xyz="1 0 0"/>
-  			<origin xyz="0 -0.00407 0.04983" rpy="0.4 0 0"/>
-			<limit lower="0" upper="0.8" effort="100" velocity="100"/>
-			<mimic joint="${prefix}_j0" multiplier="0.4" offset="0"/>
-		</joint>
-		-->
-		<joint name="${prefix}_j1" type="fixed">
+                        <parent link="${prefix}_link_0"/>
+                        <child link="${prefix}_link_1"/>
+                        <axis xyz="1 0 0"/>
+                        <origin xyz="0 -0.00407 0.04983" rpy="0.4 0 0"/>
+                        <limit lower="0" upper="0.8" effort="100" velocity="100"/>
+                        <mimic joint="${prefix}_j0" multiplier="0.4" offset="0"/>
+                </joint>
+                -->
+                <joint name="${prefix}_j1" type="fixed">
                         <parent link="${prefix}_link_0"/>
                         <child link="${prefix}_link_1"/>
@@ -100,5 +120,5 @@
                         <!--<mimic joint="${prefix}_j0" multiplier="0.4" offset="0"/>-->
                 </joint>
-		<!-- end of joint list -->
-	</xacro:macro>
+                <!-- end of joint list -->
+        </xacro:macro>
 </robot>

Commit message: Format files using xmllint

File: thor_vt_hand_description/urdf/vt_finger_tud.urdf.xacro (robot description, xacro)
@@ -1,2 +1,3 @@
+<?xml version="1.0"?>
 <!--
 parameters:
@@ -6,51 +7,51 @@
 -->
 <robot xmlns:xacro="http://ros.org/wiki/xacro">
-        <xacro:include filename="$(find thor_mang_description)/urdf/helper_macros.urdf.xacro.xml" />
-        <xacro:include filename="$(find thor_mang_description)/urdf/constants.xacro" />
-        <xacro:macro name="vt_finger_tud_macro" params="prefix reflect">
-                <!-- link list -->
-                <link name="${prefix}_link_0">
-                        <visual>
-                                <origin xyz="0 0 0" rpy="0 0 0"/>
-                                <geometry>
-                                        <mesh filename="package://thor_vt_hand_description/meshes/collision/${prefix}_link_0.stl" />
-                                </geometry>
-                                <material name="green">
-                                        <color rgba="0 1 0 1"/>
-                                </material>
-                        </visual>
-                        <collision>
-                                <origin xyz="0 0 0" rpy="0 ${M_PI*0.5} 0"/>
-                                <geometry>
-                                    <cylinder length="0.02" radius="0.017" />
-                                  </geometry>
-                                <material name="yellow">
-                                        <color rgba="0 1 1 1"/>
-                                </material>
-                        </collision>
-                        <collision>
-                                <origin xyz="0 0 0.02" rpy="0 0 0"/>
-                                <geometry>
-                                    <cylinder length="0.04" radius="0.008" />
-                                  </geometry>
-                                <material name="yellow"/>
-                        </collision>
-                        <collision>
-                                <origin xyz="0 -0.00407 0.042" rpy="0 ${M_PI*0.5} 0"/>
-                                <geometry>
-                                    <cylinder length="0.02" radius="0.014" />
-                                  </geometry>
-                                <material name="yellow">
-                                        <color rgba="0 1 1 1"/>
-                                </material>
-                        </collision>
-            <!-- WARNING: INERTIA NOT CORRECT -->
-            <inertial>
-                <origin xyz="${reflect*0.2e-03} 0.92e-03 21.11e-03" rpy="0 0 0"/>
-                <mass value="0.1"/>
-                <inertia ixx="21.39e-06" ixy="${reflect*(-0.39e-06)}" ixz="${reflect*0.71e-06}" iyy="18.98e-06" iyz="-1.36e-06" izz="4.73e-06" />
-            </inertial>
-                </link>
-                    <gazebo reference="${prefix}_link_0">
+  <xacro:include filename="$(find thor_mang_description)/urdf/helper_macros.urdf.xacro.xml"/>
+  <xacro:include filename="$(find thor_mang_description)/urdf/constants.xacro"/>
+  <xacro:macro name="vt_finger_tud_macro" params="prefix reflect">
+    <!-- link list -->
+    <link name="${prefix}_link_0">
+      <visual>
+        <origin xyz="0 0 0" rpy="0 0 0"/>
+        <geometry>
+          <mesh filename="package://thor_vt_hand_description/meshes/collision/${prefix}_link_0.stl"/>
+        </geometry>
+        <material name="green">
+          <color rgba="0 1 0 1"/>
+        </material>
+      </visual>
+      <collision>
+        <origin xyz="0 0 0" rpy="0 ${M_PI*0.5} 0"/>
+        <geometry>
+          <cylinder length="0.02" radius="0.017"/>
+        </geometry>
+        <material name="yellow">
+          <color rgba="0 1 1 1"/>
+        </material>
+      </collision>
+      <collision>
+        <origin xyz="0 0 0.02" rpy="0 0 0"/>
+        <geometry>
+          <cylinder length="0.04" radius="0.008"/>
+        </geometry>
+        <material name="yellow"/>
+      </collision>
+      <collision>
+        <origin xyz="0 -0.00407 0.042" rpy="0 ${M_PI*0.5} 0"/>
+        <geometry>
+          <cylinder length="0.02" radius="0.014"/>
+        </geometry>
+        <material name="yellow">
+          <color rgba="0 1 1 1"/>
+        </material>
+      </collision>
+      <!-- WARNING: INERTIA NOT CORRECT -->
+      <inertial>
+        <origin xyz="${reflect*0.2e-03} 0.92e-03 21.11e-03" rpy="0 0 0"/>
+        <mass value="0.1"/>
+        <inertia ixx="21.39e-06" ixy="${reflect*(-0.39e-06)}" ixz="${reflect*0.71e-06}" iyy="18.98e-06" iyz="-1.36e-06" izz="4.73e-06"/>
+      </inertial>
+    </link>
+    <gazebo reference="${prefix}_link_0">
       <mu1>1.1</mu1>
       <mu2>1.1</mu2>
@@ -62,21 +63,21 @@
       <!--<material>Gazebo/FlatBlack</material>-->
     </gazebo>
-                <link name="${prefix}_link_1">
-                        <visual>
-                                <origin xyz="0 0 0" rpy="0 0 0"/>
-                                <geometry>
-                                        <mesh filename="package://thor_vt_hand_description/meshes/collision/${prefix}_link_1.stl" />
-                                </geometry>
-                                <material name="green"/>
-                        </visual>
-                        <collision>
-                                <origin xyz="-0.002 0.007 0.018" rpy="0 0 0"/>
-                                <geometry>
-                                    <cylinder length="0.05" radius="0.008" />
-                                  </geometry>
-                                <material name="yellow"/>
-                        </collision>
-            <!-- WARNING: INERTIA NOT CORRECT -->
-            <!--
+    <link name="${prefix}_link_1">
+      <visual>
+        <origin xyz="0 0 0" rpy="0 0 0"/>
+        <geometry>
+          <mesh filename="package://thor_vt_hand_description/meshes/collision/${prefix}_link_1.stl"/>
+        </geometry>
+        <material name="green"/>
+      </visual>
+      <collision>
+        <origin xyz="-0.002 0.007 0.018" rpy="0 0 0"/>
+        <geometry>
+          <cylinder length="0.05" radius="0.008"/>
+        </geometry>
+        <material name="yellow"/>
+      </collision>
+      <!-- WARNING: INERTIA NOT CORRECT -->
+      <!--
             <inertial>
                 <origin xyz="${reflect*-0.99e-03} -4.42e-03 11.82e-03" rpy="0 0 0"/>
@@ -85,9 +86,9 @@
             </inertial>
             -->
-            <xacro:inertial_cuboid__with_pose_macro mass="0.05" x_length="0.01" y_length="0.015" z_length="0.04">
-              <origin xyz="0.0 0.005 0.02" rpy="0 0 0"/>
-            </xacro:inertial_cuboid__with_pose_macro>
-                </link>
-                    <gazebo reference="${prefix}_link_1">
+      <xacro:inertial_cuboid__with_pose_macro mass="0.05" x_length="0.01" y_length="0.015" z_length="0.04">
+        <origin xyz="0.0 0.005 0.02" rpy="0 0 0"/>
+      </xacro:inertial_cuboid__with_pose_macro>
+    </link>
+    <gazebo reference="${prefix}_link_1">
       <mu1>1.1</mu1>
       <mu2>1.1</mu2>
@@ -99,8 +100,8 @@
       <!--<material>Gazebo/FlatBlack</material>-->
     </gazebo>
-                <!-- end of link list -->
-                <!-- joint list -->
-                <!-- WARNING: UPPER LIMIT NOT CORRECT/IGNORED WHILE USING MIMIC JOINT TYPE -->
-                <!--
+    <!-- end of link list -->
+    <!-- joint list -->
+    <!-- WARNING: UPPER LIMIT NOT CORRECT/IGNORED WHILE USING MIMIC JOINT TYPE -->
+    <!--
                 <joint name="${prefix}_j1" type="revolute">
                         <parent link="${prefix}_link_0"/>
@@ -112,13 +113,13 @@
                 </joint>
                 -->
-                <joint name="${prefix}_j1" type="fixed">
-                        <parent link="${prefix}_link_0"/>
-                        <child link="${prefix}_link_1"/>
-                        <axis xyz="1 0 0"/>
-                        <origin xyz="0 -0.00407 0.04983" rpy="0.4 0 0"/>
-                        <limit lower="0" upper="0.8" effort="100" velocity="100"/>
-                        <!--<mimic joint="${prefix}_j0" multiplier="0.4" offset="0"/>-->
-                </joint>
-                <!-- end of joint list -->
-        </xacro:macro>
+    <joint name="${prefix}_j1" type="fixed">
+      <parent link="${prefix}_link_0"/>
+      <child link="${prefix}_link_1"/>
+      <axis xyz="1 0 0"/>
+      <origin xyz="0 -0.00407 0.04983" rpy="0.4 0 0"/>
+      <limit lower="0" upper="0.8" effort="100" velocity="100"/>
+      <!--<mimic joint="${prefix}_j0" multiplier="0.4" offset="0"/>-->
+    </joint>
+    <!-- end of joint list -->
+  </xacro:macro>
 </robot>

Commit message: renamed finger controllers, added friction and deleted vt_hand_tester

File: thor_vt_hand_description/urdf/vt_finger_tud.urdf.xacro (robot description, xacro)
@@ -104,15 +104,5 @@
     <!-- joint list -->
     <!-- WARNING: UPPER LIMIT NOT CORRECT/IGNORED WHILE USING MIMIC JOINT TYPE -->
-    <!--
-                <joint name="${prefix}_j1" type="revolute">
-                        <parent link="${prefix}_link_0"/>
-                        <child link="${prefix}_link_1"/>
-                        <axis xyz="1 0 0"/>
-                        <origin xyz="0 -0.00407 0.04983" rpy="0.4 0 0"/>
-                        <limit lower="0" upper="0.8" effort="100" velocity="100"/>
-                        <mimic joint="${prefix}_j0" multiplier="0.4" offset="0"/>
-                </joint>
-                -->
-    <joint name="${prefix}_j1" type="fixed">
+    <joint name="${prefix}_j1" type="revolute">
       <parent link="${prefix}_link_0"/>
       <child link="${prefix}_link_1"/>
@@ -120,5 +110,6 @@
       <origin xyz="0 -0.00407 0.04983" rpy="0.4 0 0"/>
       <limit lower="0" upper="0.8" effort="100" velocity="100"/>
-      <!--<mimic joint="${prefix}_j0" multiplier="0.4" offset="0"/>-->
+      <mimic joint="${prefix}_j0" multiplier="0.4" offset="0"/>
+      <dynamics friction="${joint_friction}" damping="${joint_damping}" />
     </joint>
     <!-- end of joint list -->

File: thor_vt_hand_description/urdf/vt_hand_tud.urdf.xacro (robot description, xacro)
@@ -4,4 +4,6 @@
   <!--<xacro:include filename="$(find thor_vt_hand_description)/urdf/vt_finger_tud.urdf.xacro"/>-->
   <xacro:include filename="$(find thor_vt_hand_description)/urdf/vt_finger_tud_single_link.urdf.xacro"/>
+  <xacro:property name="joint_friction" value="0.1" />
+  <xacro:property name="joint_damping" value="0.0" />
   <xacro:macro name="vt_hand_tud_macro" params="parent prefix reflect *origin">
     <xacro:vt_finger_tud_macro prefix="${prefix}_f1" reflect="${reflect*(-1)}"/>
@@ -55,5 +57,5 @@
       <origin xyz="${reflect*0.036} 0.0361 0.0596" rpy="-1.315 0 0"/>
       <limit lower="0" upper="2.685" effort="10" velocity="10"/>
-      <!--<dynamics damping="0.1"/>-->
+      <dynamics friction="${joint_friction}" damping="${joint_damping}" />
     </joint>
     <joint name="${prefix}_f0_j0" type="revolute">
@@ -63,5 +65,5 @@
       <origin xyz="${reflect*-0.0355} 0.0361 0.0596" rpy="-1.315 0 0"/>
       <limit lower="0" upper="2.685" effort="10" velocity="10"/>
-      <!--<dynamics damping="0.1"/>-->
+      <dynamics friction="${joint_friction}" damping="${joint_damping}" />
     </joint>
     <!-- end of joint list -->
