Commit message: Updated link names to match original robot

File: thor_vt_hand_description/hands/vt_hand_ghost.urdf.xacro (robot description, xacro)
@@ -5,5 +5,5 @@
        xmlns:xacro="http://playerstage.sourceforge.net/gazebo/xmlschema/#interface"
        name="vt_hand_ghost" >
-  <link name="$(arg name_short)_hand">
+  <link name="$(arg name_short)_arm_wr_p_link">
     <inertial>
         <mass value="0.1" />
@@ -25,5 +25,5 @@
   </link>
   <xacro:include filename="$(find thor_vt_hand_description)/urdf/vt_hand_tud.urdf.xacro.xml" />
-  <vt_hand_tud_macro parent="$(arg name_short)_hand" prefix="$(arg name_short)" reflect="$(arg reflect)" >
+  <vt_hand_tud_macro parent="$(arg name_short)_arm_wr_p_link" prefix="$(arg name_short)" reflect="$(arg reflect)" >
     <origin xyz="0 0 0" rpy="0 0 0"/>
   </vt_hand_tud_macro>
